File: Ratgo_TW/Ratgo_TW.kicad_pcb (KiCad board)
At the start: 2 copper layers, 3 parts, among them U1 ESP8266EX, U2 ESP-WROOM-02

Commit message: latest with all footprints
Parts:
- removed U1: ESP8266EX, Package_DFN_QFN:QFN-32-1EP_5x5mm_P0.5mm_EP3.45x3.45mm
- removed U2: ESP-WROOM-02, RF_Module:ESP-WROOM-02
- added C1: 1uF, Capacitor_SMD:C_0805_2012Metric, F.Cu at (87.8, 129.3)
- added C2: 100nF, Capacitor_SMD:C_0805_2012Metric, F.Cu at (87.8, 132.3)
- added C3: 1uF, Capacitor_SMD:C_0805_2012Metric, F.Cu at (87.8, 135.3)
- added C4: 10uF, Capacitor_SMD:C_0805_2012Metric, F.Cu at (87.8, 138.4)
- added J1: 10118193-0001LF, Ratgo2:AMPHENOL_10118193-0001LF, F.Cu at (55.7, 162.5)
- added J2: Screw_Terminal_01x03, Ratgo2:TB006-508-03BE, F.Cu at (95.3, 111.0)
- added Q1: 2N7002, Package_TO_SOT_SMD:SOT-23, F.Cu at (99.1, 155.0)
- added Q2: AO3400A, Package_TO_SOT_SMD:SOT-23, F.Cu at (78.9, 159.4)
- added R1: 10k, Resistor_SMD:R_0805_2012Metric, F.Cu at (83.3, 129.3)
- added R2: 10k, Resistor_SMD:R_0805_2012Metric, F.Cu at (83.3, 132.2)
- added R3: 10k, Resistor_SMD:R_0805_2012Metric, F.Cu at (83.3, 135.2)
- added R4: 10k, Resistor_SMD:R_0805_2012Metric, F.Cu at (83.3, 138.2)
- added R5: 10k, Resistor_SMD:R_0805_2012Metric, F.Cu at (83.3, 141.1)
- added R6: 10k, Resistor_SMD:R_0805_2012Metric, F.Cu at (83.3, 144.1)
- added R7: 10k, Resistor_SMD:R_0805_2012Metric, F.Cu at (83.3, 147.0)
- added SW1: SW_RST, EasyEDA:SW-SMD_4P-L6.2-W6.2-P4.00-LS6.8, F.Cu at (34.5, 137.1)
- added SW2: SW_FLASH, EasyEDA:SW-SMD_4P-L6.2-W6.2-P4.00-LS6.8, F.Cu at (19.0, 151.5)
- added U3: AP2112K-3.3, Package_TO_SOT_SMD:SOT-23-5, F.Cu at (99.4, 145.1)
- added U4: ESP-12F, RF_Module:ESP-12E, F.Cu at (58.5, 139.0)
- J3: value ~ -> Conn_01x06; footprint Connector_Phoenix_SPT:BCH-508hs-3 -> Ratgo2:METZ-CONNECT_PR20206VBNN
- moved J3 66.2 mm to (62.6, 107.5)
Connections:
- J3 pad 1: Net-(J3-Pin_1) -> unconnected-(J3-Pad1)
Routing:
- net Net-(U4-GPIO3/RXD): track 98.0 -> 0.00 mm
- net Net-(U4-GPIO1/TXD): track 43.8 -> 0.00 mm, vias 2 -> 0
